File: kicad/arduino-farm.sch (KiCad schematic (older format))
At the start: 42 parts, among them J1 Screw_Terminal_01x06, J2 Screw_Terminal_01x06, J3 Screw_Terminal_01x06, J4 Screw_Terminal_01x06, J5 Screw_Terminal_01x06, J6 Screw_Terminal_01x06, K1 SANYOU_SRD_Form_C, Q1 IRLZ34N, Q2 IRLZ34N, Q3 IRLZ34N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

Commit message: m
Parts:
- D2, D3, D4, D5, D6, D7: value DIODE -> 1N4007
Changed lines of the file:
@@
 EESchema Schematic File Version 4
-LIBS:arduino-farm-cache
 EELAYER 30 0
 EELAYER END
@@
 P 3850 1500
 F 0 "D2" V 3896 1372 50  0000 R CNN
-F 1 "DIODE" V 3805 1372 50  0000 R CNN
+F 1 "1N4007" V 3805 1372 50  0000 R CNN
 F 2 "Diode_THT:D_DO-41_SOD81_P7.62mm_Horizontal" H 3850 1500 50  0001 C CNN
 F 3 "~" H 3850 1500 50  0001 C CNN
@@
 P 5750 1500
 F 0 "D3" V 5796 1372 50  0000 R CNN
-F 1 "DIODE" V 5705 1372 50  0000 R CNN
+F 1 "1N4007" V 5705 1372 50  0000 R CNN
 F 2 "Diode_THT:D_DO-41_SOD81_P7.62mm_Horizontal" H 5750 1500 50  0001 C CNN
 F 3 "~" H 5750 1500 50  0001 C CNN
@@
 P 7700 1500
 F 0 "D4" V 7746 1372 50  0000 R CNN
-F 1 "DIODE" V 7655 1372 50  0000 R CNN
+F 1 "1N4007" V 7655 1372 50  0000 R CNN
 F 2 "Diode_THT:D_DO-41_SOD81_P7.62mm_Horizontal" H 7700 1500 50  0001 C CNN
 F 3 "~" H 7700 1500 50  0001 C CNN
@@
 P 3850 3350
 F 0 "D5" V 3896 3222 50  0000 R CNN
-F 1 "DIODE" V 3805 3222 50  0000 R CNN
+F 1 "1N4007" V 3805 3222 50  0000 R CNN
 F 2 "Diode_THT:D_DO-41_SOD81_P7.62mm_Horizontal" H 3850 3350 50  0001 C CNN
 F 3 "~" H 3850 3350 50  0001 C CNN
@@
 P 5750 3350
 F 0 "D6" V 5796 3222 50  0000 R CNN
-F 1 "DIODE" V 5705 3222 50  0000 R CNN
+F 1 "1N4007" V 5705 3222 50  0000 R CNN
 F 2 "Diode_THT:D_DO-41_SOD81_P7.62mm_Horizontal" H 5750 3350 50  0001 C CNN
 F 3 "~" H 5750 3350 50  0001 C CNN
@@
 P 7700 3350
 F 0 "D7" V 7746 3222 50  0000 R CNN
-F 1 "DIODE" V 7655 3222 50  0000 R CNN
+F 1 "1N4007" V 7655 3222 50  0000 R CNN
 F 2 "Diode_THT:D_DO-41_SOD81_P7.62mm_Horizontal" H 7700 3350 50  0001 C CNN
 F 3 "~" H 7700 3350 50  0001 C CNN
